File: Hardware/V3/Waveform_Generator/Waveform_Generator.kicad_pcb (KiCad board)
At the start: 2 copper layers, 160 x 100 mm, 108 parts, among them J101 DIN41612_02x32_AC, J201 Wave_Out, J401 SWD, J402 Address, K201 G6K-2, Q201 BSS138, Q401 BSS138, Q402 BSS138, U201 AD9833xRM, U202 OPA2196xD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

Commit message: Code Update Implement full code for Waveform Generator Small doc update Readme Update
Changed lines of the file:
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@@
     (property "Sheetname" "Analog")
     (attr smd)
-    (fp_text reference "U204" (at 0 -2.6 -90) (layer "F.SilkS")
+    (fp_text reference "U204" (at -2.794 3.81) (layer "F.SilkS")
       (effects (font (size 1 1) (thickness 0.15)))
     )
