File: Hardware/V3/Waveform_Generator/analog.kicad_sch (KiCad schematic)
At the start: 58 parts, among them J201 Wave_Out, K201 G6K-2, Q201 BSS138, U201 AD9833xRM, U202 OPA2196xD, U203 LM7171xIM, U204 VCA822, X201 25MHz

Commit message: Code Update Implement full code for Waveform Generator Small doc update Readme Update
Parts:
- R218: value 200 -> 1k
- R220: value 1k -> 200
Changed lines of the file:
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@@
     (in_bom yes) (on_board yes) (fields_autoplaced)
     (property "Reference" "R220" (id 0) (at 213.36 48.6242 90))
-    (property "Value" "1k" (id 1) (at 213.36 51.1611 90))
+    (property "Value" "200" (id 1) (at 213.36 51.1611 90))
     (property "Footprint" "Resistor_SMD:R_0805_2012Metric" (id 2) (at 213.36 55.118 90)
       (effects (font (size 1.27 1.27)) hide)
@@
     (in_bom yes) (on_board yes) (fields_autoplaced)
     (property "Reference" "R218" (id 0) (at 194.31 21.9542 90))
-    (property "Value" "200" (id 1) (at 194.31 24.4911 90))
+    (property "Value" "1k" (id 1) (at 194.31 24.4911 90))
     (property "Footprint" "Resistor_SMD:R_0805_2012Metric" (id 2) (at 194.31 28.448 90)
       (effects (font (size 1.27 1.27)) hide)
