File: Hardware/V3/Power_SMPS/Power_SMPS.kicad_pcb (KiCad board)
At the start: 2 copper layers, 160 x 100 mm, 117 parts, among them J101 DIN41612_02x32_AC, J102 Conn_01x02, J301 Address, J302 SWD, K101 ADW11, Q101 BSS138, Q201 BD140, Q202 TIP3055, Q301 BSS138, Q302 BSS138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

Commit message: SMPS Schematic and PCB Bugfix
Parts:
- K101: footprint Relay_THT:Relay_SPST_Panasonic_JW1_FormA -> eigene:JS 05 MN KT
- moved K101 2.86 mm to (78.9, 66.4)
Connections:
- J102 pad 1: Net-(K101-Pad3) -> Net-(J102-Pad1)
Routing:
- net Net-(D101-Pad2): track 0.01 -> 6.78 mm
- added copper zone on F.Cu, net Net-(J102-Pad1)
- removed copper zone on F.Cu, net Net-(K101-Pad3)
Changed lines of the file:
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@@
   (net 113 "unconnected-(U402-Pad8)")
   (net 114 "Net-(D101-Pad2)")
-  (net 115 "Net-(K101-Pad3)")
+  (net 115 "Net-(J102-Pad1)")
   (footprint "Resistor_SMD:R_0805_2012Metric" (layer "F.Cu")
     (at 201.42 90.174 -90)
@@
     (fp_line (start -1.27 -1.27) (end 0.635 -1.27) (layer "F.Fab") (width 0.1))
     (pad "1" thru_hole rect (at 0 0) (size 1.7 1.7) (drill 1) (layers *.Cu *.Mask)
-      (net 115 "Net-(K101-Pad3)") (pinfunction "Pin_1") (pintype "passive"))
+      (net 115 "Net-(J102-Pad1)") (pinfunction "Pin_1") (pintype "passive"))
     (pad "2" thru_hole oval (at 0 2.54) (size 1.7 1.7) (drill 1) (layers *.Cu *.Mask)
       (net 2 "GND") (pinfunction "Pin_2") (pintype "passive"))
@@
     )
   )
-  (footprint "Relay_THT:Relay_SPST_Panasonic_JW1_FormA" (layer "F.Cu")
-    (at 80.0825 68.9805 -90)
-    (descr "Panasonic Relay SPST, http://www3.panasonic.biz/ac/e_download/control/relay/power/catalog/mech_eng_jw.pdf?via=ok")
-    (tags "Panasonic Relay SPST")
+  (footprint "eigene:JS 05 MN KT" (layer "F.Cu")
+    (at 78.915 66.367 -90)
     (property "Sheetfile" "Power_SMPS.kicad_sch")
     (property "Sheetname" "")
     (attr through_hole)
-    (fp_text reference "K101" (at 12.1 -11.5 90) (layer "F.SilkS")
+    (fp_text reference "K101" (at 0 -0.5 -90 unlocked) (layer "F.SilkS")
       (effects (font (size 1 1) (thickness 0.15)))
     )
-    (fp_text value "ADW11" (at 12.1 3.9 90) (layer "F.Fab")
+    (fp_text value "ADW11" (at 0 1 -90 unlocked) (layer "F.Fab")
       (effects (font (size 1 1) (thickness 0.15)))
     )
-    (fp_text user "${REFERENCE}" (at 12 -3.75 90) (layer "F.Fab")
-      (effects (font (size 1 1) (thickness 0.15)))
-    )
-    (fp_line (start 26 -10.3) (end -2.8 -10.3) (layer "F.SilkS") (width 0.12))
-    (fp_line (start -1 -4.15) (end -1 -3.45) (layer "F.SilkS") (width 0.12))
-    (fp_line (start -3.04 2.94) (end -3.04 0.6) (layer "F.SilkS") (width 0.12))
-    (fp_line (start -2.8 2.7) (end 26 2.7) (layer "F.SilkS") (width 0.12))
-    (fp_line (start 0.2 -4.15) (end -1 -4.15) (layer "F.SilkS") (width 0.12))
-    (fp_line (start -0.2 -3.45) (end -0.6 -4.15) (layer "F.SilkS") (width 0.12))
-    (fp_line (start -1 -3.45) (end 0.2 -3.45) (layer "F.SilkS") (width 0.12))
-    (fp_line (start -0.7 2.94) (end -3.04 2.94) (layer "F.SilkS") (width 0.12))
-    (fp_line (start 0.2 -3.45) (end 0.2 -4.15) (layer "F.SilkS") (width 0.12))
-    (fp_line (start -2.8 -10.3) (end -2.8 2.7) (layer "F.SilkS") (width 0.12))
-    (fp_line (start 26 2.7) (end 26 -10.3) (layer "F.SilkS") (width 0.12))
-    (fp_line (start -2.95 2.85) (end 26.15 2.85) (layer "F.CrtYd") (width 0.05))
-    (fp_line (start 26.15 2.85) (end 26.15 -10.45) (layer "F.CrtYd") (width 0.05))
-    (fp_line (start 26.15 -10.45) (end -2.95 -10.45) (layer "F.CrtYd") (width 0.05))
-    (fp_line (start -2.95 -10.45) (end -2.95 2.85) (layer "F.CrtYd") (width 0.05))
-    (fp_line (start -1 2.6) (end -2.7 1) (layer "F.Fab") (width 0.12))
-    (fp_line (start -1 2.6) (end 25.9 2.6) (layer "F.Fab") (width 0.1))
-    (fp_line (start -3.04 2.94) (end -3.04 0.6) (layer "F.Fab") (width 0.1))
-    (fp_line (start -0.4 -1.55) (end -0.4 -6.05) (layer "F.Fab") (width 0.1))
-    (fp_line (start -0.7 2.94) (end -3.04 2.94) (layer "F.Fab") (width 0.1))
-    (fp_line (start 25.9 -10.2) (end -2.7 -10.2) (layer "F.Fab") (width 0.1))
-    (fp_line (start 25.9 2.6) (end 25.9 -10.2) (layer "F.Fab") (width 0.1))
-    (fp_line (start -2.7 -10.2) (end -2.7 1) (layer "F.Fab") (width 0.1))
-    (pad "1" thru_hole rect (at 0 0) (size 2.5 2.5) (drill 1.5) (layers *.Cu *.Mask)
+    (fp_line (start 1 -6) (end 1 -4) (layer "F.SilkS") (width 0.12))
+    (fp_line (start 29 0) (end 29 -10) (layer "F.SilkS") (width 0.12))
+    (fp_line (start 0 -6) (end 1 -6) (layer "F.SilkS") (width 0.12))
+    (fp_line (start 0 -10) (end 0 0) (layer "F.SilkS") (width 0.12))
+    (fp_line (start 29 -10) (end 0 -10) (layer "F.SilkS") (width 0.12))
+    (fp_line (start 20 0) (end 29 0) (layer "F.SilkS") (width 0.12))
+    (fp_line (start 1 -4) (end 0 -4) (layer "F.SilkS") (width 0.12))
+    (fp_line (start 0 0) (end 20 0) (layer "F.SilkS") (width 0.12))
+    (fp_line (start 0.35 0) (end 0.35 -1.19) (layer "User.1") (width 0.12))
+    (pad "1" thru_hole circle (at 2.5 -1.19) (size 2 2) (drill 1.2) (layers *.Cu *.Mask)
       (net 24 "+5V") (pintype "passive"))
-    (pad "4" thru_hole oval (at 23.5 0) (size 2.5 2.5) (drill 1.5) (layers *.Cu *.Mask))
-    (pad "6" thru_hole oval (at 20 -7.6) (size 2.5 2.5) (drill 1.5) (layers *.Cu *.Mask)
+    (pad "3" thru_hole circle (at 21.4 -1.19) (size 2 2) (drill 1.2) (layers *.Cu *.Mask)
+      (net 115 "Net-(J102-Pad1)") (pintype "passive"))
+    (pad "5" thru_hole circle (at 26.4 -8.81) (size 2 2) (drill 1.2) (layers *.Cu *.Mask)
+      (net 59 "/SMPS/VOut") (pintype "passive"))
+    (pad "6" thru_hole circle (at 2.5 -8.82) (size 2 2) (drill 1.2) (layers *.Cu *.Mask)
       (net 114 "Net-(D101-Pad2)") (pintype "passive"))
-    (pad "8" thru_hole oval (at 0 -7.6) (size 2.5 2.5) (drill 1.5) (layers *.Cu *.Mask))
-    (model "${KICAD6_3DMODEL_DIR}/Relay_THT.3dshapes/Relay_SPST_Panasonic_JW1_FormA.wrl"
-      (offset (xyz 0 0 0))
-      (scale (xyz 1 1 1))
-      (rotate (xyz 0 0 0))
-    )
   )
   (footprint "Package_TO_SOT_SMD:SOT-223-3_TabPin2" (layer "F.Cu")
@@
   (segment (start 175.768 93.472) (end 187.579 81.661) (width 0.2) (layer "F.Cu") (net 87))
   (segment (start 164.6905 94.762) (end 165.899686 94.762) (width 0.2) (layer "F.Cu") (net 87))
-  (segment (start 87.655 62.1515) (end 87.6625 62.159) (width 0.2) (layer "F.Cu") (net 114))
+  (segment (start 87.655 62.1515) (end 87.627 62.1795) (width 0.3) (layer "F.Cu") (net 114))
+  (segment (start 87.627 62.1795) (end 87.627 64.516) (width 0.3) (layer "F.Cu") (net 114))
+  (segment (start 87.655 62.1515) (end 87.6625 62.159) (width 0.3) (layer "F.Cu") (net 114))
+  (segment (start 87.627 68.759) (end 87.735 68.867) (width 0.3) (layer "F.Cu") (net 114))
+  (segment (start 87.627 64.516) (end 87.627 68.759) (width 0.3) (layer "F.Cu") (net 114))
   (zone (net 1) (net_name "+24V") (layer "F.Cu") (hatch edge 0.508)
     (priority 1)
@@
     )
   )
-  (zone (net 115) (net_name "Net-(K101-Pad3)") (layer "F.Cu") (hatch edge 0.508)
+  (zone (net 115) (net_name "Net-(J102-Pad1)") (layer "F.Cu") (hatch edge 0.508)
     (priority 1)
     (connect_pads yes (clearance 0.254))
@@
         (xy 82.55 99.568)
         (xy 77.47 99.568)
-        (xy 77.47 89.916)
-        (xy 82.55 89.916)
+        (xy 77.47 85.598)
+        (xy 82.55 85.598)
       )
     )
@@
     (polygon
       (pts
-        (xy 94.742 92.456)
-        (xy 85.344 92.456)
+        (xy 94.742 95.504)
+        (xy 85.344 95.504)
         (xy 85.344 85.344)
         (xy 94.742 85.344)
@@
         (xy 100.838 113.792)
         (xy 88.392 113.792)
-        (xy 88.392 94.488)
-        (xy 94.742 94.488)
+        (xy 88.392 96.52)
+        (xy 94.742 96.52)
         (xy 94.742 85.344)
         (xy 100.838 85.344)
