File: Hardware/V3/Power_SMPS/smps.kicad_sch (KiCad schematic)
At the start: 35 parts, among them Q201 BD140, Q202 TIP3055, U201 LM2902, U202 TL494

Commit message: PCB Update
Parts:
- R209: value 12k -> 5k6
- R219: value 12k -> 8k2
Other:
- note removed: "Widerstand einbauen! 100R oda so"
Changed lines of the file:
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@@
     (stroke (width 0) (type default) (color 0 0 0 0))
   )
-  (text "Widerstand einbauen! 100R oda so" (at 227.33 149.86 0)
-    (effects (font (size 1.27 1.27)) (justify left bottom))
-  )
   (text "Current Sense Amplifier" (at 157.48 71.12 0)
-    (effects (font (size 1.27 1.27)) (justify left bottom))
-  )
-  (text "Widerstand einbauen! 100R oda so" (at 177.8 121.92 0)
     (effects (font (size 1.27 1.27)) (justify left bottom))
   )
@@
     (in_bom yes) (on_board yes) (fields_autoplaced)
     (property "Reference" "R209" (id 0) (at 151.13 112.1242 90))
-    (property "Value" "12k" (id 1) (at 151.13 114.6611 90))
+    (property "Value" "5k6" (id 1) (at 151.13 114.6611 90))
     (property "Footprint" "Resistor_SMD:R_0805_2012Metric" (id 2) (at 151.13 118.618 90)
       (effects (font (size 1.27 1.27)) hide)
@@
       (effects (font (size 1.27 1.27)) (justify right))
     )
-    (property "Value" "12k" (id 1) (at 202.438 152.8322 0)
+    (property "Value" "8k2" (id 1) (at 202.438 152.8322 0)
       (effects (font (size 1.27 1.27)) (justify right))
     )
